File: Lighting.kicad_sch (KiCad schematic)
At the start: 17 parts, among them J11 436500212, J6 436500212, J7 436500212, J8 436500312, Q1 FDS8949, U4 SN74LVC1G125DBV

Commit message: Completed V1.0 draft layout - pending review
Parts:
- removed C17, C18, C19, C21: 47uF, Capacitor_SMD:CP_Elec_5x5.4, symbol Device:C_Polarized

Commit message: Work-in-progress: Layout
Parts:
- removed J6, J7: 436500212, butterfly-footprint-libs:436500212, symbol Connector_Generic:Conn_01x02
- removed unit 2 of Q1
- removed R14: 100k, Resistor_SMD:R_0402_1005Metric_Pad0.72x0.64mm_HandSolder, symbol Device:R
- added C38: 1uF, Capacitor_SMD:C_0805_2012Metric, symbol Device:C
- added C39: 4.7uF, Capacitor_Tantalum_SMD:CP_EIA-3216-10_Kemet-I, symbol Device:C_Polarized
- added C40: 220nF, Capacitor_SMD:C_0402_1005Metric, symbol Device:C
- added D10: MBR0530, Diode_SMD:D_SOD-123, symbol Diode:MBR0530
- added D11, D12, D13, D14: LED, butterfly-footprint-libs:GW Q9LR33, symbol Device:LED
- added J5: 694106301002, butterfly-footprint-libs:694106301002, symbol butterfly-schematic-libs:694106301002
- added L1: 10uH, Inductor_SMD:L_1210_3225Metric, symbol Device:L
- added U13: TPS61165DBV, Package_TO_SOT_SMD:SOT-23-6, symbol Driver_LED:TPS61165DBV
- R13: value 100 -> 0.6; footprint Resistor_SMD:R_0402_1005Metric_Pad0.72x0.64mm_HandSolder -> Resistor_SMD:R_1206_3216Metric; JLC C25076 -> C407230
Connections:
- net +12V: now also J5.1
- net GND: now also R13.2, C38.2, C39.2, C40.2, U13.4 (GND)
- net INTERNAL_LED_PWM: now also U13.2 (CTRL); no longer R13.1
- net at Q1.7 (D), Q1.8 (D): now also J5.2, J5.3
- new net: D10.2 (A), L1.2, U13.3 (SW)
- new net: C40.1, U13.5 (COMP)
- new net: D14.1 (K), R13.1, U13.6 (FB)
- new net: D11.1 (K), D12.2 (A)
- new net: C38.1, D10.1 (K), D11.2 (A)
- new net: D12.1 (K), D13.2 (A)
- new net: D13.1 (K), D14.2 (A)
- new net +5VA: C39.1, L1.1, U13.1 (VIN)
Other:
- note added: "*SHOULD NOT USE USB POWER."
- note added: "I=300mA"
- note added: "V_{trip}=0.2V (typical)"
- moved on the sheet: C20, C22, C23, J11, J8, Q1A, R11, R12, U4
