File: MCU-ATega328P.kicad_sch (KiCad schematic)
At the start: 32 parts, among them J1 1054500101, J2 AVR-ISP-6, J4 Conn_01x04, SW1 RESET, U1 ATmega328P-M, U2 FT231XQ, Y1 16MHz

Commit message: Completed V1.0 draft layout - pending review
Parts:
- C6: footprint Capacitor_SMD:CP_Elec_4x5.4 -> Capacitor_Tantalum_SMD:CP_EIA-3216-10_Kemet-I; JLC C3348 -> C7174
- C7: footprint Capacitor_SMD:CP_Elec_4x5.4 -> Capacitor_Tantalum_SMD:CP_EIA-3216-10_Kemet-I; JLC C3355 -> C7187
- J2: symbol Connector:AVR-ISP-6 -> Connector_Generic:Conn_02x03_Odd_Even
- Y1: MPN CSTNE16M0VH3C000R0 -> (none)
Connections:
- net MISO: now also J2.1 (Pin_1); no longer J2.4 (MOSI)
- net MOSI: now also J2.4 (Pin_4); no longer J2.1 (MISO)
