File: Porto-Butterfly.kicad_pcb (KiCad board)
At the start: 4 copper layers, 120 x 50 mm, 106 parts, among them J1 1054500101, J10 436500212, J11 436500212, J2 AVR-ISP-6, J3 436500212, J4 Conn_01x04, J6 436500212, J7 436500212, J8 436500312, J9 436500212, Q1 FDS8949, Q4 NCE3080KA, Q5 NCE3080KA, SW1 RESET, U1 ATmega328P-M, U2 FT231XQ, U3 VEML6030, U4 SN74LVC1G125DBV, U5 TPS5450DDAR, U6 STHS34PF80TR, U7 AMS1117-3.3, Y1 16MHz

Commit message: Work-in-progress: Layout
Parts:
- removed C14, C8: 100nF, Capacitor_SMD:C_0402_1005Metric
- removed C9: 10uF, Capacitor_SMD:C_0402_1005Metric
- removed the H1 at (332.6, 74.2)
- removed the H2 at (332.6, 85.0)
- removed the H3 at (332.6, 95.8)
- removed the H4 at (332.6, 106.5)
- removed J6, J7: 436500212, butterfly-footprint-libs:436500212
- removed R14: 100k, Resistor_SMD:R_0402_1005Metric_Pad0.72x0.64mm_HandSolder
- removed R17, R18, R19, R20, R21: 10k, Resistor_SMD:R_0402_1005Metric_Pad0.72x0.64mm_HandSolder
- removed R8: 10R, Resistor_SMD:R_0402_1005Metric_Pad0.72x0.64mm_HandSolder
- removed TP1, TP2, TP3, TP4, TP5: TestPoint, TestPoint:TestPoint_Pad_D1.5mm
- removed U3: VEML6030, butterfly-footprint-libs:VEML6030
- removed U6: STHS34PF80TR, butterfly-footprint-libs:STHS34PF80TR
- added C17: 4.7uF, Capacitor_SMD:C_0402_1005Metric, B.Cu at (144.4, 97.8)
- added C18: 100nF, Capacitor_SMD:C_0402_1005Metric, B.Cu at (144.4, 98.9)
- added C19: 100nF, Capacitor_SMD:C_0402_1005Metric, F.Cu at (110.8, 118.6)
- added C21: 100nF, Capacitor_SMD:C_0402_1005Metric, B.Cu at (144.3, 107.5)
- added C24: 100nF, Capacitor_SMD:C_0402_1005Metric, B.Cu at (150.8, 103.2)
- added C37: 100nF, Capacitor_SMD:C_0402_1005Metric, B.Cu at (149.6, 98.9)
- added C38: 1uF, Capacitor_SMD:C_0805_2012Metric, B.Cu at (168.0, 82.9)
- added C39: 4.7uF, Capacitor_Tantalum_SMD:CP_EIA-3216-10_Kemet-I, B.Cu at (168.5, 88.9)
- added C40: 220nF, Capacitor_SMD:C_0402_1005Metric, B.Cu at (171.6, 92.4)
- added D10: MBR0530, Diode_SMD:D_SOD-123, B.Cu at (171.5, 81.9)
- added D11: LED, butterfly-footprint-libs:GW Q9LR33, B.Cu at (147.0, 89.0)
- added D12: LED, butterfly-footprint-libs:GW Q9LR33, B.Cu at (132.0, 104.0)
- added D13: LED, butterfly-footprint-libs:GW Q9LR33, B.Cu at (147.0, 119.0)
- added D14: LED, butterfly-footprint-libs:GW Q9LR33, B.Cu at (162.0, 104.0)
- added J5: 694106301002, butterfly-footprint-libs:694106301002, F.Cu at (170.0, 120.9)
- added L1: 10uH, Inductor_SMD:L_1210_3225Metric, B.Cu at (171.6, 84.9)
- added R28: 10k, Resistor_SMD:R_0402_1005Metric_Pad0.72x0.64mm_HandSolder, B.Cu at (142.2, 103.2)
- added R29: 10k, Resistor_SMD:R_0402_1005Metric_Pad0.72x0.64mm_HandSolder, B.Cu at (142.2, 98.9)
- added R30: 200k, Resistor_SMD:R_0402_1005Metric, F.Cu at (109.7, 118.6)
- added R31: 2.2k, Resistor_SMD:R_0402_1005Metric_Pad0.72x0.64mm_HandSolder, F.Cu at (118.5, 117.9)
- added R32: 2.2k, Resistor_SMD:R_0402_1005Metric_Pad0.72x0.64mm_HandSolder, F.Cu at (118.5, 115.2)
- added R33: 0, Resistor_SMD:R_0402_1005Metric, B.Cu at (145.3, 109.5)
- added R34: 0, Resistor_SMD:R_0402_1005Metric, B.Cu at (147.5, 109.5)
- added R35: 0, Resistor_SMD:R_0402_1005Metric, B.Cu at (146.4, 109.5)
- added R36: 0, Resistor_SMD:R_0402_1005Metric, B.Cu at (148.6, 109.5)
- added R37: 3.3M, Resistor_SMD:R_0603_1608Metric, B.Cu at (152.1, 98.6)
- added U10: TMP117AIDRVR, Package_SON:WSON-6-1EP_2x2mm_P0.65mm_EP1x1.6mm, B.Cu at (147.0, 107.0)
- added U11: AS7331, butterfly-footprint-libs:AS7331, B.Cu at (149.2, 100.0)
- added U13: TPS61165DBV, Package_TO_SOT_SMD:SOT-23-6, B.Cu at (171.6, 88.9)
- added U8: VL53L0CXV0DH, Sensor_Distance:ST_VL53L1x, B.Cu at (143.2, 101.0)
- added U9: LSF0102DCTR, butterfly-footprint-libs:DCT0008A_M, F.Cu at (114.6, 117.0)
- R13: value 100 -> 0.6; footprint Resistor_SMD:R_0402_1005Metric_Pad0.72x0.64mm_HandSolder -> Resistor_SMD:R_1206_3216Metric; moved to B.Cu
- moved U7 27.8 mm to (166.2, 99.9)
- moved C35 27.0 mm to (165.6, 106.2)
- moved C34 25.9 mm to (165.6, 105.0)
- moved R27 25.8 mm to (183.2, 124.5), turned to -90 degrees
- moved R15 25.8 mm to (189.9, 124.5), turned to -90 degrees
- moved D9 25.0 mm to (185.0, 124.5), turned to -90 degrees
- moved C10 24.7 mm to (179.8, 96.8), turned to 180 degrees
- moved D4 23.7 mm to (188.0, 124.5), turned to -90 degrees
- moved C33 20.1 mm to (170.4, 102.5), turned to 90 degrees
- moved D8 19.5 mm to (187.4, 114.0), turned to 0 degrees
- moved R9 16.6 mm to (191.0, 93.2)
- moved C28 15.7 mm to (204.2, 108.2), turned to 0 degrees
- moved Q1 14.8 mm to (170.4, 110.7)
- moved R10 14.5 mm to (191.0, 94.4), turned to 0 degrees
- moved C27 14.5 mm to (199.6, 109.9), turned to 180 degrees
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Connections:
- net Net-(D4-A) renamed +5VA
- Q1 pad 3: GND -> (no net)
- Q1 pad 4: Net-(Q1B-G) -> (no net)
- Q1 pad 5: Net-(J7-Pin_2) -> (no net)
- Q1 pad 6: Net-(J7-Pin_2) -> (no net)
- R13 pad 1: /Lighting/INTERNAL_LED_PWM -> Net-(D14-K)
- R13 pad 2: Net-(Q1B-G) -> GND
Routing:
- net GND: track 0.00 -> 34.7 mm, vias 0 -> 74
- net +5VA: track 0.00 -> 18.5 mm
- net /Power Supply/VSENSE: track 0.00 -> 6.95 mm
- net +5V: track 0.00 -> 5.56 mm
- net Net-(U1-XTAL1/PB6): track 0.00 -> 4.00 mm
- net Net-(U5-BOOT): track 0.00 -> 3.57 mm
- net Net-(U1-XTAL2/PB7): track 0.00 -> 3.50 mm
- net +3.3V: track 0.00 -> 3.17 mm
- net Net-(D3-K): track 0.00 -> 1.83 mm
- added copper zone on F.Cu, net /Power Supply/12VIN
- added copper zone on F.Cu, net GND
- added copper zone on In1.Cu, net GND
- added copper zone on F.Cu, net Net-(D3-K)
Other:
- board text added: "B.Cu ="
- board text added: "EXT. LED"
- board text added: "F.Cu ="
- board text added: "IN1.Cu = GND"
- board text added: "IN2.Cu ="
- board text removed: "EXTERNAL LED POWER"
