File: Porto-Butterfly.kicad_sch (KiCad schematic)
At the start: 5 parts, among them J3 436500212

Commit message: Work-in-progress: Layout
Connections:
- no-connect marks 0 -> 2
Other:
- sheet Sensors ports: added ~{INT_LUX}; removed ~{INT_HP}, ~{INT_IR}
Changed lines of the file:
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@@
 	(title_block
 		(title "Porto - Butterfly")
-		(date "2025-02-20")
+		(date "2025-02-23")
 		(rev "v2.0")
 	)
+	(no_connect
+		(at 237.49 166.37)
+	)
+	(no_connect
+		(at 237.49 132.08)
+	)
 	(wire
 		(pts
@@
 	(wire
 		(pts
+			(xy 234.95 132.08) (xy 237.49 132.08)
+		)
+		(stroke
+			(width 0)
+			(type default)
+		)
+	)
+	(wire
+		(pts
+			(xy 234.95 166.37) (xy 237.49 166.37)
+		)
+		(stroke
+			(width 0)
+			(type default)
+		)
+	)
+	(wire
+		(pts
 			(xy 284.48 201.93) (xy 246.38 201.93)
 		)
@@
 		(pts
 			(xy 259.08 149.86) (xy 259.08 177.8)
-		)
-		(stroke
-			(width 0)
-			(type default)
-		)
-	)
-	(wire
-		(pts
-			(xy 234.95 132.08) (xy 284.48 132.08)
 		)
 		(stroke
@@
 			)
 		)
-		(pin "~{INT_IR}" output
+		(pin "~{INT_LUX}" output
 			(at 284.48 129.54 180)
 			(effects
 				(font
-					(size 1.27 1.27)
-				)
-				(justify left)
-			)
-		)
-		(pin "~{INT_HP}" output
-			(at 284.48 132.08 180)
-			(effects
-				(font
