File: Power-Supply.kicad_sch (KiCad schematic)
At the start: 29 parts, among them U5 TPS5450DDAR, U7 AMS1117-3.3

Commit message: Completed V1.0 draft layout - pending review
Parts:
- removed C24: 4.7uF, Capacitor_SMD:CP_Elec_4x5.4, symbol Device:C_Polarized
- added C36: 4.7uF, Capacitor_Tantalum_SMD:CP_EIA-3216-10_Kemet-I, symbol Device:C_Polarized
- C11: footprint Capacitor_SMD:CP_Elec_4x5.4 -> Capacitor_Tantalum_SMD:CP_EIA-3216-10_Kemet-I; JLC C3355 -> C7187
- C30: footprint Capacitor_SMD:CP_Elec_4x5.4 -> Capacitor_Tantalum_SMD:CP_EIA-3216-10_Kemet-I; JLC C3348 -> C7174
Connections:
- net 12VIN: now also C36.1
- net GND: now also C36.2

Commit message: Work-in-progress: Layout
Connections:
- net +5VA: now reaches C27.1, C28.1, D4.2 (A), D8.2 (A), L2.2, R9.1
Changed lines of the file:
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@@
 	(title_block
 		(title "Porto - Butterfly")
-		(date "2025-02-20")
+		(date "2025-02-23")
 		(rev "v2.0")
 	)
@@
 		(pts
 			(xy 273.05 101.6) (xy 273.05 99.06)
+		)
+		(stroke
+			(width 0)
+			(type default)
+		)
+	)
+	(wire
+		(pts
+			(xy 273.05 93.98) (xy 273.05 99.06)
 		)
 		(stroke
@@
 				(bold yes)
 			)
+		)
+	)
+	(label "12VIN"
+		(at 127 99.06 0)
+		(fields_autoplaced yes)
+		(effects
+			(font
+				(size 1.27 1.27)
+			)
+			(justify left bottom)
 		)
 	)
@@
 					(unit 1)
 				)
+			)
+		)
+	)
+	(symbol
+		(lib_id "power:+5VA")
+		(at 273.05 93.98 0)
+		(unit 1)
+		(exclude_from_sim no)
+		(in_bom yes)
+		(on_board yes)
+		(dnp no)
+		(fields_autoplaced yes)
+		(property "Reference" "#PWR079"
+			(at 273.05 97.79 0)
+			(effects
+				(font
+					(size 1.27 1.27)
+				)
+				(hide yes)
+			)
+		)
+		(property "Value" "+5VA"
+			(at 273.05 88.9 0)
+			(effects
+				(font
+					(size 1.27 1.27)
+				)
+			)
+		)
+		(property "Footprint" ""
+			(at 273.05 93.98 0)
+			(effects
+				(font
+					(size 1.27 1.27)
+				)
+				(hide yes)
+			)
+		)
+		(property "Datasheet" ""
+			(at 273.05 93.98 0)
+			(effects
+				(font
+					(size 1.27 1.27)
+				)
+				(hide yes)
+			)
+		)
+		(property "Description" "Power symbol creates a global label with name \"+5VA\""
+			(at 273.05 93.98 0)
+			(effects
+				(font
+					(size 1.27 1.27)
+				)
+				(hide yes)
+			)
+		)
+		(pin "1"
+		)
+		(instances
+			(project ""
+				(path "/e3f039c6-0c07-4c61-9e22-bac2658b40f2/92a536ec-3a01-4a5d-a060-cc0f59bf8839"
+					(reference "#PWR079")
+					(unit 1)
+				)
