File: Sensors.kicad_sch (KiCad schematic)
At the start: 11 parts, among them U3 VEML6030, U6 STHS34PF80TR

Commit message: Work-in-progress: Layout
Parts:
- removed C14, C8: 100nF, Capacitor_SMD:C_0402_1005Metric, symbol Device:C
- removed C9: 10uF, Capacitor_SMD:C_0402_1005Metric, symbol Device:C
- removed R17, R18, R19, R20, R21: 10k, Resistor_SMD:R_0402_1005Metric_Pad0.72x0.64mm_HandSolder, symbol Device:R
- removed R8: 10R, Resistor_SMD:R_0402_1005Metric_Pad0.72x0.64mm_HandSolder, symbol Device:R
- removed U3: VEML6030, butterfly-footprint-libs:VEML6030, symbol butterfly-schematic-libs:VEML6030
- removed U6: STHS34PF80TR, butterfly-footprint-libs:STHS34PF80TR, symbol butterfly-schematic-libs:STHS34PF80TR
- added C17: 4.7uF, Capacitor_SMD:C_0402_1005Metric, symbol Device:C
- added C18, C19, C21, C24, C37: 100nF, Capacitor_SMD:C_0402_1005Metric, symbol Device:C
- added R28, R29: 10k, Resistor_SMD:R_0402_1005Metric_Pad0.72x0.64mm_HandSolder, symbol Device:R
- added R30: 200k, Resistor_SMD:R_0402_1005Metric, symbol Device:R
- added R31, R32: 2.2k, Resistor_SMD:R_0402_1005Metric_Pad0.72x0.64mm_HandSolder, symbol Device:R
- added R33, R34, R35, R36: 0, Resistor_SMD:R_0402_1005Metric, symbol Device:R
- added R37: 3.3M, Resistor_SMD:R_0603_1608Metric, symbol Device:R
- added U10: TMP117AIDRVR, Package_SON:WSON-6-1EP_2x2mm_P0.65mm_EP1x1.6mm, symbol Sensor_Temperature:TMP117xxDRV
- added U11: AS7331, butterfly-footprint-libs:AS7331, symbol butterfly-schematic-libs:AS7331
- added U8: VL53L0CXV0DH, Sensor_Distance:ST_VL53L1x, symbol Sensor_Distance:VL53L0CXV0DH1
- added U9: LSF0102DCTR, butterfly-footprint-libs:DCT0008A_M, symbol butterfly-schematic-libs:LSF0102DCTR
Connections:
- net +3.3V: now also C17.1, C18.2, C24.1, C37.1, R31.1, R32.1, U11.14 (VDDA), U11.7 (VDDD), U8.1 (AVDDVCSEL), U8.11 (AVDD), U9.2 (V_{REFA})
- net GND: now also C17.2, C18.1, C19.2, C21.1, C24.2, C37.2, R36.1, R37.2, U10.2 (GND), U11.1 (VSSA), U11.10 (A1), U11.11 (VSSA), U11.12 (VSSA), U11.15 (VSSA), U11.16 (VSSA), U11.2 (VSSA), U11.3 (A0), U11.6 (VSSD), U8.12 (GND), U8.2 (AVSSVCSEL), U8.3 (GND), U8.4 (GND), U8.6 (GND), U9.1 (GND)
- net SCL: now also R34.1, U10.1 (SCL), U9.6 (B1)
- net SDA: now also R33.1, U10.6 (SDA), U9.5 (B2)
- new net: C19.1, R30.2, U9.7 (V_{REFB}), U9.8 (EN)
- new net: R29.2, U8.5 (XSHUT)
- new net: R33.2, R34.2, R35.2, R36.2, U10.4 (ADD0)
- new net: R37.1, U11.13 (REXT)
- new net +5V: C21.2, R28.1, R29.1, R30.1, R35.1, U10.5 (V+)
- new net SCL_3V3: R31.2, U11.4 (SCL), U8.10 (SCL), U9.3 (A1)
- new net SDA_3V3: R32.2, U11.5 (SDA), U8.9 (SDA), U9.4 (A2)
- new net ~{INT_LUX}: R28.2, U8.7 (GPIO1)
- no-connect marks 0 -> 3
Other:
- note added: "LOGIC LEVEL SHIFTER 5V->3.3V"
- note added: "Populate only one."
- note added: "TEMPERATURE SENSOR"
- note added: "TOF SENSOR"
- note added: "UV SENSOR"
